Commit message: change xacro

File: imu_description/urdf/imu.xacro (robot description, xacro)
@@ -7,7 +7,7 @@
       <origin rpy="${roll} ${pitch} ${yaw}" xyz="${x} ${y} ${z}"/>
       <parent link="${parent}"/>
-      <child link="${name}_link"/>
+      <child link="${name}"/>
     </joint>
-    <link name="${name}_link">
+    <link name="${name}">
       <visual>
         <geometry>
@@ -39,5 +39,5 @@
     </link>
     <!-- imu -->
-    <gazebo reference="${name}_link">
+    <gazebo reference="${name}">
       <gravity>true</gravity>
       <sensor name="${name}_sensor" type="imu">
